File: design/8x8_module.kicad_sch (KiCad schematic)
At the start: 68 parts, among them U6 MAX7219

Commit message: Added some more sheets, new board layout
Parts:
- removed D10, D18, D26, D34, D42, D50, D58: Green, LED_THT:LED_D3.0mm_Clear, symbol Device:LED_Small
- added D3, D4, D5, D6, D7, D8, D9: Green, LED_THT:LED_D5.0mm, symbol Device:LED_Small
- D10: renamed from D3; footprint LED_THT:LED_D3.0mm_Clear -> LED_THT:LED_D5.0mm
- D11, D12, D13, D14, D15, D16, D17, D19, D2, D20, D21, D22, D23, D24, D25, D27, D28, D29, D30, D31, D32, D33, D35, D36, D37, D38, D39, D40, D41, D43, D44, D45, D46, D47, D48, D49, D51, D52, D53, D54, D55, D56, D57, D59, D60, D61, D62, D63, D64, D65: footprint LED_THT:LED_D3.0mm_Clear -> LED_THT:LED_D5.0mm
- D18: renamed from D4; footprint LED_THT:LED_D3.0mm_Clear -> LED_THT:LED_D5.0mm
- D26: renamed from D5; footprint LED_THT:LED_D3.0mm_Clear -> LED_THT:LED_D5.0mm
- D34: renamed from D6; footprint LED_THT:LED_D3.0mm_Clear -> LED_THT:LED_D5.0mm
- D42: renamed from D7; footprint LED_THT:LED_D3.0mm_Clear -> LED_THT:LED_D5.0mm
- D50: renamed from D8; footprint LED_THT:LED_D3.0mm_Clear -> LED_THT:LED_D5.0mm
- D58: renamed from D9; footprint LED_THT:LED_D3.0mm_Clear -> LED_THT:LED_D5.0mm
- renumbered C12 to C3, C13 to C4, R10 to R2, U6 to U2
Connections:
- net 1: now also D3.2 (A), D4.2 (A), D5.2 (A), D6.2 (A), D7.2 (A), D8.2 (A), D9.2 (A); no longer D19.2 (A), D35.2 (A), D36.2 (A), D37.2 (A)
- net 2: now also D12.2 (A), D13.2 (A), D14.2 (A), D15.2 (A), D16.2 (A), D17.2 (A); no longer D20.2 (A), D21.2 (A), D38.2 (A), D39.2 (A), D40.2 (A), D41.2 (A)
- net 3: now also D19.2 (A), D20.2 (A), D21.2 (A), D24.2 (A), D25.2 (A); no longer D12.2 (A), D43.2 (A), D44.2 (A), D45.2 (A)
- net 4: now also D27.2 (A), D28.2 (A), D29.2 (A), D30.2 (A), D31.2 (A), D32.2 (A), D33.2 (A); no longer D13.2 (A), D24.2 (A), D25.2 (A), D46.2 (A), D47.2 (A), D48.2 (A), D49.2 (A)
- net 5: now also D35.2 (A), D36.2 (A), D37.2 (A), D38.2 (A), D39.2 (A), D40.2 (A), D41.2 (A); no longer D14.2 (A), D27.2 (A), D51.2 (A), D52.2 (A), D53.2 (A)
- net 6: now also D43.2 (A), D44.2 (A), D45.2 (A), D46.2 (A), D47.2 (A), D48.2 (A), D49.2 (A); no longer D15.2 (A), D28.2 (A), D29.2 (A), D54.2 (A), D55.2 (A), D56.2 (A), D57.2 (A)
- net 7: now also D51.2 (A), D52.2 (A), D53.2 (A), D54.2 (A), D55.2 (A), D56.2 (A), D57.2 (A); no longer D16.2 (A), D30.2 (A), D31.2 (A), D59.2 (A), D60.2 (A), D61.2 (A)
- net 8: now also D59.2 (A), D60.2 (A), D61.2 (A); no longer D17.2 (A), D32.2 (A), D33.2 (A)
- net B: now also D19.1 (K), D27.1 (K), D35.1 (K), D43.1 (K), D51.1 (K), D59.1 (K), D3.1 (K); no longer D12.1 (K), D13.1 (K), D14.1 (K), D15.1 (K), D16.1 (K), D17.1 (K)
- net C: now also D12.1 (K), D36.1 (K), D44.1 (K), D52.1 (K), D60.1 (K), D4.1 (K); no longer D22.1 (K), D24.1 (K), D30.1 (K), D32.1 (K)
- net D: now also D13.1 (K), D37.1 (K), D45.1 (K), D53.1 (K), D61.1 (K), D5.1 (K); no longer D19.1 (K), D23.1 (K), D25.1 (K), D27.1 (K), D31.1 (K), D33.1 (K)
- net E: now also D14.1 (K), D22.1 (K), D30.1 (K), D6.1 (K)
- net F: now also D15.1 (K), D23.1 (K), D31.1 (K), D7.1 (K); no longer D35.1 (K), D43.1 (K), D51.1 (K), D59.1 (K)
- net G: now also D16.1 (K), D24.1 (K), D32.1 (K), D8.1 (K); no longer D36.1 (K), D44.1 (K), D52.1 (K), D60.1 (K)
- net H: now also D17.1 (K), D25.1 (K), D33.1 (K), D9.1 (K); no longer D37.1 (K), D45.1 (K), D53.1 (K), D61.1 (K)

Commit message: layout mostly done, schematic is done, need to generate new updated pdf
Parts:
- D10: renamed from D3; footprint LED_THT:LED_D5.0mm -> LED_SMD:LED_0805_2012Metric_Pad1.15x1.40mm_HandSolder
- D11, D2, D20, D29, D38, D47, D56, D65: footprint LED_THT:LED_D5.0mm -> LED_SMD:LED_0805_2012Metric_Pad1.15x1.40mm_HandSolder
- D12: renamed from D19; footprint LED_THT:LED_D5.0mm -> LED_SMD:LED_0805_2012Metric_Pad1.15x1.40mm_HandSolder
- D13: renamed from D27; footprint LED_THT:LED_D5.0mm -> LED_SMD:LED_0805_2012Metric_Pad1.15x1.40mm_HandSolder
- D14: renamed from D35; footprint LED_THT:LED_D5.0mm -> LED_SMD:LED_0805_2012Metric_Pad1.15x1.40mm_HandSolder
- D15: renamed from D43; footprint LED_THT:LED_D5.0mm -> LED_SMD:LED_0805_2012Metric_Pad1.15x1.40mm_HandSolder
- D16: renamed from D51; footprint LED_THT:LED_D5.0mm -> LED_SMD:LED_0805_2012Metric_Pad1.15x1.40mm_HandSolder
- D17: renamed from D59; footprint LED_THT:LED_D5.0mm -> LED_SMD:LED_0805_2012Metric_Pad1.15x1.40mm_HandSolder
- D18: renamed from D4; footprint LED_THT:LED_D5.0mm -> LED_SMD:LED_0805_2012Metric_Pad1.15x1.40mm_HandSolder
- D19: renamed from D12; footprint LED_THT:LED_D5.0mm -> LED_SMD:LED_0805_2012Metric_Pad1.15x1.40mm_HandSolder
- D21: renamed from D28; footprint LED_THT:LED_D5.0mm -> LED_SMD:LED_0805_2012Metric_Pad1.15x1.40mm_HandSolder
- D22: renamed from D36; footprint LED_THT:LED_D5.0mm -> LED_SMD:LED_0805_2012Metric_Pad1.15x1.40mm_HandSolder
- D23: renamed from D44; footprint LED_THT:LED_D5.0mm -> LED_SMD:LED_0805_2012Metric_Pad1.15x1.40mm_HandSolder
- D24: renamed from D52; footprint LED_THT:LED_D5.0mm -> LED_SMD:LED_0805_2012Metric_Pad1.15x1.40mm_HandSolder
- D25: renamed from D60; footprint LED_THT:LED_D5.0mm -> LED_SMD:LED_0805_2012Metric_Pad1.15x1.40mm_HandSolder
- D26: renamed from D5; footprint LED_THT:LED_D5.0mm -> LED_SMD:LED_0805_2012Metric_Pad1.15x1.40mm_HandSolder
- D27: renamed from D13; footprint LED_THT:LED_D5.0mm -> LED_SMD:LED_0805_2012Metric_Pad1.15x1.40mm_HandSolder
- D28: renamed from D21; footprint LED_THT:LED_D5.0mm -> LED_SMD:LED_0805_2012Metric_Pad1.15x1.40mm_HandSolder
- D3: renamed from D10; footprint LED_THT:LED_D5.0mm -> LED_SMD:LED_0805_2012Metric_Pad1.15x1.40mm_HandSolder
- D30: renamed from D37; footprint LED_THT:LED_D5.0mm -> LED_SMD:LED_0805_2012Metric_Pad1.15x1.40mm_HandSolder
- D31: renamed from D45; footprint LED_THT:LED_D5.0mm -> LED_SMD:LED_0805_2012Metric_Pad1.15x1.40mm_HandSolder
- D32: renamed from D53; footprint LED_THT:LED_D5.0mm -> LED_SMD:LED_0805_2012Metric_Pad1.15x1.40mm_HandSolder
- D33: renamed from D61; footprint LED_THT:LED_D5.0mm -> LED_SMD:LED_0805_2012Metric_Pad1.15x1.40mm_HandSolder
- D34: renamed from D6; footprint LED_THT:LED_D5.0mm -> LED_SMD:LED_0805_2012Metric_Pad1.15x1.40mm_HandSolder
- D35: renamed from D14; footprint LED_THT:LED_D5.0mm -> LED_SMD:LED_0805_2012Metric_Pad1.15x1.40mm_HandSolder
- D36: renamed from D22; footprint LED_THT:LED_D5.0mm -> LED_SMD:LED_0805_2012Metric_Pad1.15x1.40mm_HandSolder
- D37: renamed from D30; footprint LED_THT:LED_D5.0mm -> LED_SMD:LED_0805_2012Metric_Pad1.15x1.40mm_HandSolder
- D39: renamed from D46; footprint LED_THT:LED_D5.0mm -> LED_SMD:LED_0805_2012Metric_Pad1.15x1.40mm_HandSolder
- D4: renamed from D18; footprint LED_THT:LED_D5.0mm -> LED_SMD:LED_0805_2012Metric_Pad1.15x1.40mm_HandSolder
- D40: renamed from D54; footprint LED_THT:LED_D5.0mm -> LED_SMD:LED_0805_2012Metric_Pad1.15x1.40mm_HandSolder
- D41: renamed from D62; footprint LED_THT:LED_D5.0mm -> LED_SMD:LED_0805_2012Metric_Pad1.15x1.40mm_HandSolder
- D42: renamed from D7; footprint LED_THT:LED_D5.0mm -> LED_SMD:LED_0805_2012Metric_Pad1.15x1.40mm_HandSolder
- D43: renamed from D15; footprint LED_THT:LED_D5.0mm -> LED_SMD:LED_0805_2012Metric_Pad1.15x1.40mm_HandSolder
- D44: renamed from D23; footprint LED_THT:LED_D5.0mm -> LED_SMD:LED_0805_2012Metric_Pad1.15x1.40mm_HandSolder
- D45: renamed from D31; footprint LED_THT:LED_D5.0mm -> LED_SMD:LED_0805_2012Metric_Pad1.15x1.40mm_HandSolder
- D46: renamed from D39; footprint LED_THT:LED_D5.0mm -> LED_SMD:LED_0805_2012Metric_Pad1.15x1.40mm_HandSolder
- D48: renamed from D55; footprint LED_THT:LED_D5.0mm -> LED_SMD:LED_0805_2012Metric_Pad1.15x1.40mm_HandSolder
- D49: renamed from D63; footprint LED_THT:LED_D5.0mm -> LED_SMD:LED_0805_2012Metric_Pad1.15x1.40mm_HandSolder
- D5: renamed from D26; footprint LED_THT:LED_D5.0mm -> LED_SMD:LED_0805_2012Metric_Pad1.15x1.40mm_HandSolder
- D50: renamed from D8; footprint LED_THT:LED_D5.0mm -> LED_SMD:LED_0805_2012Metric_Pad1.15x1.40mm_HandSolder
- D51: renamed from D16; footprint LED_THT:LED_D5.0mm -> LED_SMD:LED_0805_2012Metric_Pad1.15x1.40mm_HandSolder
- D52: renamed from D24; footprint LED_THT:LED_D5.0mm -> LED_SMD:LED_0805_2012Metric_Pad1.15x1.40mm_HandSolder
- D53: renamed from D32; footprint LED_THT:LED_D5.0mm -> LED_SMD:LED_0805_2012Metric_Pad1.15x1.40mm_HandSolder
- D54: renamed from D40; footprint LED_THT:LED_D5.0mm -> LED_SMD:LED_0805_2012Metric_Pad1.15x1.40mm_HandSolder
- D55: renamed from D48; footprint LED_THT:LED_D5.0mm -> LED_SMD:LED_0805_2012Metric_Pad1.15x1.40mm_HandSolder
- D57: renamed from D64; footprint LED_THT:LED_D5.0mm -> LED_SMD:LED_0805_2012Metric_Pad1.15x1.40mm_HandSolder
- D58: renamed from D9; footprint LED_THT:LED_D5.0mm -> LED_SMD:LED_0805_2012Metric_Pad1.15x1.40mm_HandSolder
- D59: renamed from D17; footprint LED_THT:LED_D5.0mm -> LED_SMD:LED_0805_2012Metric_Pad1.15x1.40mm_HandSolder
- D6: renamed from D34; footprint LED_THT:LED_D5.0mm -> LED_SMD:LED_0805_2012Metric_Pad1.15x1.40mm_HandSolder
- D60: renamed from D25; footprint LED_THT:LED_D5.0mm -> LED_SMD:LED_0805_2012Metric_Pad1.15x1.40mm_HandSolder
- D61: renamed from D33; footprint LED_THT:LED_D5.0mm -> LED_SMD:LED_0805_2012Metric_Pad1.15x1.40mm_HandSolder
- D62: renamed from D41; footprint LED_THT:LED_D5.0mm -> LED_SMD:LED_0805_2012Metric_Pad1.15x1.40mm_HandSolder
- D63: renamed from D49; footprint LED_THT:LED_D5.0mm -> LED_SMD:LED_0805_2012Metric_Pad1.15x1.40mm_HandSolder
- D64: renamed from D57; footprint LED_THT:LED_D5.0mm -> LED_SMD:LED_0805_2012Metric_Pad1.15x1.40mm_HandSolder
- D7: renamed from D42; footprint LED_THT:LED_D5.0mm -> LED_SMD:LED_0805_2012Metric_Pad1.15x1.40mm_HandSolder
- D8: renamed from D50; footprint LED_THT:LED_D5.0mm -> LED_SMD:LED_0805_2012Metric_Pad1.15x1.40mm_HandSolder
- D9: renamed from D58; footprint LED_THT:LED_D5.0mm -> LED_SMD:LED_0805_2012Metric_Pad1.15x1.40mm_HandSolder
- renumbered R2 to R4
