File: design/PSUs.kicad_sch (KiCad schematic)
At the start: 3 parts, among them U2 TLV75533PDBV

Commit message: Added some more sheets, new board layout
Parts:
- renumbered C2 to C1, C1 to C2, U2 to U1

Commit message: layout mostly done, schematic is done, need to generate new updated pdf
Parts:
- renumbered C2 to C1, C1 to C2
Changed lines of the file:
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@@
 		(dnp no)
 		(fields_autoplaced yes)
-		(property "Reference" "C2"
+		(property "Reference" "C1"
 			(at 161.29 89.5412 0)
 			(effects
@@
 			(project ""
 				(path "/e36fbef8-3f03-40ce-b8c1-50d21e162c91/e2792bac-e585-4209-b69f-ff39bd7e7a6c"
-					(reference "C2")
+					(reference "C1")
 					(unit 1)
 				)
@@
 		(on_board yes)
 		(dnp no)
-		(property "Reference" "#PWR09"
+		(property "Reference" "#PWR010"
 			(at 158.115 88.9 0)
 			(effects
@@
 			(project ""
 				(path "/e36fbef8-3f03-40ce-b8c1-50d21e162c91/e2792bac-e585-4209-b69f-ff39bd7e7a6c"
-					(reference "#PWR09")
+					(reference "#PWR010")
 					(unit 1)
 				)
@@
 		(dnp no)
 		(fields_autoplaced yes)
-		(property "Reference" "#PWR08"
+		(property "Reference" "#PWR011"
 			(at 144.78 107.315 0)
 			(effects
@@
 			(project ""
 				(path "/e36fbef8-3f03-40ce-b8c1-50d21e162c91/e2792bac-e585-4209-b69f-ff39bd7e7a6c"
-					(reference "#PWR08")
+					(reference "#PWR011")
 					(unit 1)
 				)
@@
 		(dnp no)
 		(fields_autoplaced yes)
-		(property "Reference" "C1"
+		(property "Reference" "C2"
 			(at 133.35 92.0812 0)
 			(effects
@@
 			(project "RocketClock"
 				(path "/e36fbef8-3f03-40ce-b8c1-50d21e162c91/e2792bac-e585-4209-b69f-ff39bd7e7a6c"
-					(reference "C1")
+					(reference "C2")
 					(unit 1)
 				)
@@
 		(on_board yes)
 		(dnp no)
-		(property "Reference" "#PWR07"
+		(property "Reference" "#PWR09"
 			(at 128.27 88.9 0)
 			(effects
@@
 			(project "RocketClock"
 				(path "/e36fbef8-3f03-40ce-b8c1-50d21e162c91/e2792bac-e585-4209-b69f-ff39bd7e7a6c"
-					(reference "#PWR07")
-					(unit 1)
-				)
+					(reference "#PWR09")
+					(unit 1)
+				)
