File: design/mcu.kicad_sch (KiCad schematic)
At the start: 9 parts, among them SW1 SW_MEC_5E, U1 ESP-12F

Commit message: Added some more sheets, new board layout
Parts:
- renumbered C4 to C11, C3 to C12, C11 to C13, R3 to R10, R1 to R7, R4 to R8, R2 to R9, U1 to U5
Changed lines of the file:
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@@
 		(dnp no)
 		(fields_autoplaced yes)
-		(property "Reference" "C11"
+		(property "Reference" "C13"
 			(at 59.69 34.2962 0)
 			(effects
@@
 			(project "RocketClock"
 				(path "/e36fbef8-3f03-40ce-b8c1-50d21e162c91/31ceb4ad-97ae-4994-9156-dc2819dfe7a6"
-					(reference "C11")
+					(reference "C13")
 					(unit 1)
 				)
@@
 		(dnp no)
 		(fields_autoplaced yes)
-		(property "Reference" "R3"
+		(property "Reference" "R10"
 			(at 176.53 79.3749 0)
 			(effects
@@
 			(project "RocketClock"
 				(path "/e36fbef8-3f03-40ce-b8c1-50d21e162c91/31ceb4ad-97ae-4994-9156-dc2819dfe7a6"
-					(reference "R3")
+					(reference "R10")
 					(unit 1)
 				)
@@
 		(dnp no)
 		(fields_autoplaced yes)
-		(property "Reference" "R4"
+		(property "Reference" "R8"
 			(at 121.92 79.3749 0)
 			(effects
@@
 			(project "RocketClock"
 				(path "/e36fbef8-3f03-40ce-b8c1-50d21e162c91/31ceb4ad-97ae-4994-9156-dc2819dfe7a6"
-					(reference "R4")
+					(reference "R8")
 					(unit 1)
 				)
@@
 		(dnp no)
 		(fields_autoplaced yes)
-		(property "Reference" "#PWR01"
+		(property "Reference" "#PWR027"
 			(at 151.765 128.27 0)
 			(effects
@@
 			(project ""
 				(path "/e36fbef8-3f03-40ce-b8c1-50d21e162c91/31ceb4ad-97ae-4994-9156-dc2819dfe7a6"
-					(reference "#PWR01")
+					(reference "#PWR027")
 					(unit 1)
 				)
@@
 		(dnp no)
 		(fields_autoplaced yes)
-		(property "Reference" "C4"
+		(property "Reference" "C11"
 			(at 30.48 33.6612 0)
 			(effects
@@
 			(project "RocketClock"
 				(path "/e36fbef8-3f03-40ce-b8c1-50d21e162c91/31ceb4ad-97ae-4994-9156-dc2819dfe7a6"
-					(reference "C4")
+					(reference "C11")
 					(unit 1)
 				)
@@
 		(dnp no)
 		(fields_autoplaced yes)
-		(property "Reference" "#PWR014"
+		(property "Reference" "#PWR025"
 			(at 40.64 45.085 0)
 			(effects
@@
 			(project "RocketClock"
 				(path "/e36fbef8-3f03-40ce-b8c1-50d21e162c91/31ceb4ad-97ae-4994-9156-dc2819dfe7a6"
-					(reference "#PWR014")
+					(reference "#PWR025")
 					(unit 1)
 				)
@@
 		(on_board yes)
 		(dnp no)
-		(property "Reference" "U1"
+		(property "Reference" "U5"
 			(at 153.9083 77.47 0)
 			(effects
@@
 			(project ""
 				(path "/e36fbef8-3f03-40ce-b8c1-50d21e162c91/31ceb4ad-97ae-4994-9156-dc2819dfe7a6"
-					(reference "U1")
+					(reference "U5")
 					(unit 1)
 				)
@@
 		(dnp no)
 		(fields_autoplaced yes)
-		(property "Reference" "#PWR013"
+		(property "Reference" "#PWR024"
 			(at 40.64 34.925 0)
 			(effects
@@
 			(project "RocketClock"
 				(path "/e36fbef8-3f03-40ce-b8c1-50d21e162c91/31ceb4ad-97ae-4994-9156-dc2819dfe7a6"
-					(reference "#PWR013")
+					(reference "#PWR024")
 					(unit 1)
 				)
@@
 		(dnp no)
 		(fields_autoplaced yes)
-		(property "Reference" "#PWR02"
+		(property "Reference" "#PWR026"
 			(at 151.765 74.93 0)
 			(effects
@@
 			(project ""
 				(path "/e36fbef8-3f03-40ce-b8c1-50d21e162c91/31ceb4ad-97ae-4994-9156-dc2819dfe7a6"
-					(reference "#PWR02")
+					(reference "#PWR026")
 					(unit 1)
 				)
@@
 		(dnp no)
 		(fields_autoplaced yes)
-		(property "Reference" "C3"
+		(property "Reference" "C12"
 			(at 43.815 33.6612 0)
 			(effects
@@
 			(project ""
 				(path "/e36fbef8-3f03-40ce-b8c1-50d21e162c91/31ceb4ad-97ae-4994-9156-dc2819dfe7a6"
-					(reference "C3")
+					(reference "C12")
 					(unit 1)
 				)
@@
 		(dnp no)
 		(fields_autoplaced yes)
-		(property "Reference" "#PWR03"
+		(property "Reference" "#PWR023"
 			(at 33.655 102.87 0)
 			(effects
@@
 			(project "RocketClock"
 				(path "/e36fbef8-3f03-40ce-b8c1-50d21e162c91/31ceb4ad-97ae-4994-9156-dc2819dfe7a6"
-					(reference "#PWR03")
+					(reference "#PWR023")
 					(unit 1)
 				)
@@
 		(dnp no)
 		(fields_autoplaced yes)
-		(property "Reference" "R2"
+		(property "Reference" "R9"
 			(at 173.99 111.7599 0)
 			(effects
@@
 			(project "RocketClock"
 				(path "/e36fbef8-3f03-40ce-b8c1-50d21e162c91/31ceb4ad-97ae-4994-9156-dc2819dfe7a6"
-					(reference "R2")
+					(reference "R9")
 					(unit 1)
 				)
@@
 		(dnp no)
 		(fields_autoplaced yes)
-		(property "Reference" "R1"
+		(property "Reference" "R7"
 			(at 114.935 83.1849 0)
 			(effects
@@
 			(project ""
 				(path "/e36fbef8-3f03-40ce-b8c1-50d21e162c91/31ceb4ad-97ae-4994-9156-dc2819dfe7a6"
-					(reference "R1")
-					(unit 1)
-				)
+					(reference "R7")
+					(unit 1)
+				)

Commit message: layout mostly done, schematic is done, need to generate new updated pdf
Parts:
- removed SW1: SW_MEC_5E, Button_Switch_SMD:SW_MEC_5GSH9, symbol Switch:SW_MEC_5E
- added SW1: SW_Push, Button_Switch_SMD:SW_Push_1P1T_NO_CK_KSC6xxJ, symbol Switch:SW_Push
- renumbered C11 to C13, C12 to C14, C13 to C15, R8 to R19, R10 to R20, R7 to R21, R9 to R22, U5 to U6
Connections:
- net GND: now also SW1.1
- net ~{RST}: now also SW1.2
- net CS renamed ~{CS}
Changed lines of the file:
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@@
 	)
 	(junction
-		(at 33.655 91.44)
+		(at 40.64 31.75)
+		(diameter 0)
+		(color 0 0 0 0)
+	)
+	(junction
+		(at 40.64 38.1)
 		(diameter 0)
 		(color 0 0 0 0)
@@
 	)
 	(junction
-		(at 40.64 31.75)
-		(diameter 0)
-		(color 0 0 0 0)
-	)
-	(junction
-		(at 40.64 38.1)
-		(diameter 0)
-		(color 0 0 0 0)
-	)
-	(junction
 		(at 120.015 78.105)
 		(diameter 0)
@@
 	(wire
 		(pts
+			(xy 151.765 119.38) (xy 151.765 121.92)
+		)
+		(stroke
+			(width 0)
+			(type default)
+		)
+	)
+	(wire
+		(pts
+			(xy 151.765 73.66) (xy 151.765 71.12)
+		)
+		(stroke
+			(width 0)
+			(type default)
+		)
+	)
+	(wire
+		(pts
 			(xy 33.655 67.31) (xy 33.655 71.12)
 		)
@@
 	(wire
 		(pts
-			(xy 151.765 119.38) (xy 151.765 121.92)
-		)
-		(stroke
-			(width 0)
-			(type default)
-		)
-	)
-	(wire
-		(pts
-			(xy 151.765 73.66) (xy 151.765 71.12)
-		)
-		(stroke
-			(width 0)
-			(type default)
-		)
-	)
-	(wire
-		(pts
-			(xy 36.195 71.12) (xy 36.195 76.835)
-		)
-		(stroke
-			(width 0)
-			(type default)
-		)
-	)
-	(wire
-		(pts
 			(xy 40.64 38.1) (xy 56.515 38.1)
 		)
@@
 	(wire
 		(pts
-			(xy 33.655 76.835) (xy 33.655 71.12)
-		)
-		(stroke
-			(width 0)
-			(type default)
-		)
-	)
-	(wire
-		(pts
 			(xy 151.765 73.66) (xy 174.625 73.66)
 		)
@@
 	(wire
 		(pts
+			(xy 33.655 71.12) (xy 33.655 75.565)
+		)
+		(stroke
+			(width 0)
+			(type default)
+		)
+	)
+	(wire
+		(pts
+			(xy 29.845 71.12) (xy 33.655 71.12)
+		)
+		(stroke
+			(width 0)
+			(type default)
+		)
+	)
+	(wire
+		(pts
 			(xy 120.015 84.455) (xy 136.525 84.455)
 		)
@@
 	(wire
 		(pts
-			(xy 33.655 71.12) (xy 36.195 71.12)
-		)
-		(stroke
-			(width 0)
-			(type default)
-		)
-	)
-	(wire
-		(pts
 			(xy 113.03 78.105) (xy 113.03 81.915)
 		)
@@
 	(wire
 		(pts
-			(xy 33.655 91.44) (xy 33.655 96.52)
+			(xy 33.655 85.725) (xy 33.655 96.52)
 		)
 		(stroke
@@
 	(wire
 		(pts
-			(xy 33.655 91.44) (xy 36.195 91.44)
-		)
-		(stroke
-			(width 0)
-			(type default)
-		)
-	)
-	(wire
-		(pts
 			(xy 172.085 107.315) (xy 167.005 107.315)
 		)
@@
 	(wire
 		(pts
-			(xy 36.195 91.44) (xy 36.195 86.995)
-		)
-		(stroke
-			(width 0)
-			(type default)
-		)
-	)
-	(wire
-		(pts
 			(xy 56.515 29.21) (xy 56.515 33.02)
 		)
@@
 		)
 	)
-	(wire
-		(pts
-			(xy 33.655 86.995) (xy 33.655 91.44)
-		)
-		(stroke
-			(width 0)
-			(type default)
-		)
-	)
-	(label "CS"
-		(at 179.07 102.235 0)
+	(label "~{CS}"
+		(at 179.705 102.235 0)
 		(effects
 			(font
@@
 		)
 	)
+	(hierarchical_label "~{RST}"
+		(shape input)
+		(at 29.845 71.12 180)
+		(effects
+			(font
+				(size 1.27 1.27)
+			)
+			(justify right)
+		)
+	)
 	(hierarchical_label "+3.3V"
 		(shape input)
@@
 		)
 	)
-	(hierarchical_label "CS"
+	(hierarchical_label "~{CS}"
 		(shape input)
 		(at 193.675 102.235 0)
@@
 		(dnp no)
 		(fields_autoplaced yes)
-		(property "Reference" "C13"
+		(property "Reference" "C15"
 			(at 59.69 34.2962 0)
 			(effects
@@
 			(project "RocketClock"
 				(path "/e36fbef8-3f03-40ce-b8c1-50d21e162c91/31ceb4ad-97ae-4994-9156-dc2819dfe7a6"
-					(reference "C13")
+					(reference "C15")
 					(unit 1)
 				)
@@
 	)
 	(symbol
-		(lib_id "Switch:SW_MEC_5E")
-		(at 36.195 81.915 90)
+		(lib_id "Switch:SW_Push")
+		(at 33.655 80.645 90)
 		(unit 1)
 		(exclude_from_sim no)
@@
 		(fields_autoplaced yes)
 		(property "Reference" "SW1"
-			(at 36.83 80.6449 90)
+			(at 35.56 79.3749 90)
 			(effects
 				(font
@@
 			)
 		)
-		(property "Value" "SW_MEC_5E"
-			(at 36.83 83.1849 90)
+		(property "Value" "SW_Push"
+			(at 35.56 81.9149 90)
 			(effects
 				(font
@@
 			)
 		)
-		(property "Footprint" "Button_Switch_SMD:SW_MEC_5GSH9"
-			(at 28.575 81.915 0)
-			(effects
-				(font
-					(size 1.27 1.27)
-				)
-				(hide yes)
-			)
-		)
-		(property "Datasheet" "http://www.apem.com/int/index.php?controller=attachment&id_attachment=1371"
-			(at 28.575 81.915 0)
-			(effects
-				(font
-					(size 1.27 1.27)
-				)
-				(hide yes)
-			)
-		)
-		(property "Description" "MEC 5E single pole normally-open tactile switch"
-			(at 36.195 81.915 0)
+		(property "Footprint" "Button_Switch_SMD:SW_Push_1P1T_NO_CK_KSC6xxJ"
+			(at 28.575 80.645 0)
+			(effects
+				(font
+					(size 1.27 1.27)
+				)
+				(hide yes)
+			)
+		)
+		(property "Datasheet" "~"
+			(at 28.575 80.645 0)
+			(effects
+				(font
+					(size 1.27 1.27)
+				)
+				(hide yes)
+			)
+		)
+		(property "Description" "Push button switch, generic, two pins"
+			(at 33.655 80.645 0)
 			(effects
 				(font
@@
 		)
 		(pin "2"
-		)
-		(pin "4"
-		)
-		(pin "3"
 		)
 		(instances
@@
 		(dnp no)
 		(fields_autoplaced yes)
-		(property "Reference" "R10"
+		(property "Reference" "R20"
 			(at 176.53 79.3749 0)
 			(effects
@@
 			(project "RocketClock"
 				(path "/e36fbef8-3f03-40ce-b8c1-50d21e162c91/31ceb4ad-97ae-4994-9156-dc2819dfe7a6"
-					(reference "R10")
+					(reference "R20")
 					(unit 1)
 				)
@@
 		(dnp no)
 		(fields_autoplaced yes)
-		(property "Reference" "R8"
+		(property "Reference" "R19"
 			(at 121.92 79.3749 0)
 			(effects
@@
 			(project "RocketClock"
 				(path "/e36fbef8-3f03-40ce-b8c1-50d21e162c91/31ceb4ad-97ae-4994-9156-dc2819dfe7a6"
-					(reference "R8")
+					(reference "R19")
 					(unit 1)
 				)
@@
 		(dnp no)
 		(fields_autoplaced yes)
-		(property "Reference" "#PWR027"
+		(property "Reference" "#PWR039"
 			(at 151.765 128.27 0)
 			(effects
@@
 			(project ""
 				(path "/e36fbef8-3f03-40ce-b8c1-50d21e162c91/31ceb4ad-97ae-4994-9156-dc2819dfe7a6"
-					(reference "#PWR027")
+					(reference "#PWR039")
 					(unit 1)
 				)
@@
 		(dnp no)
 		(fields_autoplaced yes)
-		(property "Reference" "C11"
+		(property "Reference" "C13"
 			(at 30.48 33.6612 0)
 			(effects
@@
 			(project "RocketClock"
 				(path "/e36fbef8-3f03-40ce-b8c1-50d21e162c91/31ceb4ad-97ae-4994-9156-dc2819dfe7a6"
-					(reference "C11")
+					(reference "C13")
 					(unit 1)
 				)
@@
 		(dnp no)
 		(fields_autoplaced yes)
-		(property "Reference" "#PWR025"
+		(property "Reference" "#PWR036"
 			(at 40.64 45.085 0)
 			(effects
@@
 			(project "RocketClock"
 				(path "/e36fbef8-3f03-40ce-b8c1-50d21e162c91/31ceb4ad-97ae-4994-9156-dc2819dfe7a6"
-					(reference "#PWR025")
+					(reference "#PWR036")
 					(unit 1)
 				)
@@
 		(on_board yes)
 		(dnp no)
-		(property "Reference" "U5"
+		(property "Reference" "U6"
 			(at 153.9083 77.47 0)
 			(effects
@@
 			(project ""
 				(path "/e36fbef8-3f03-40ce-b8c1-50d21e162c91/31ceb4ad-97ae-4994-9156-dc2819dfe7a6"
-					(reference "U5")
+					(reference "U6")
 					(unit 1)
 				)
@@
 		(dnp no)
 		(fields_autoplaced yes)
-		(property "Reference" "#PWR024"
+		(property "Reference" "#PWR035"
 			(at 40.64 34.925 0)
 			(effects
@@
 			(project "RocketClock"
 				(path "/e36fbef8-3f03-40ce-b8c1-50d21e162c91/31ceb4ad-97ae-4994-9156-dc2819dfe7a6"
-					(reference "#PWR024")
+					(reference "#PWR035")
 					(unit 1)
 				)
@@
 		(dnp no)
 		(fields_autoplaced yes)
-		(property "Reference" "#PWR026"
+		(property "Reference" "#PWR037"
 			(at 151.765 74.93 0)
 			(effects
@@
 			(project ""
 				(path "/e36fbef8-3f03-40ce-b8c1-50d21e162c91/31ceb4ad-97ae-4994-9156-dc2819dfe7a6"
-					(reference "#PWR026")
+					(reference "#PWR037")
 					(unit 1)
 				)
@@
 		(dnp no)
 		(fields_autoplaced yes)
-		(property "Reference" "C12"
+		(property "Reference" "C14"
 			(at 43.815 33.6612 0)
 			(effects
@@
 			(project ""
 				(path "/e36fbef8-3f03-40ce-b8c1-50d21e162c91/31ceb4ad-97ae-4994-9156-dc2819dfe7a6"
-					(reference "C12")
+					(reference "C14")
 					(unit 1)
 				)
@@
 		(dnp no)
 		(fields_autoplaced yes)
-		(property "Reference" "#PWR023"
+		(property "Reference" "#PWR038"
 			(at 33.655 102.87 0)
 			(effects
@@
 			(project "RocketClock"
 				(path "/e36fbef8-3f03-40ce-b8c1-50d21e162c91/31ceb4ad-97ae-4994-9156-dc2819dfe7a6"
-					(reference "#PWR023")
+					(reference "#PWR038")
 					(unit 1)
 				)
@@
 		(dnp no)
 		(fields_autoplaced yes)
-		(property "Reference" "R9"
+		(property "Reference" "R22"
 			(at 173.99 111.7599 0)
 			(effects
@@
 			(project "RocketClock"
 				(path "/e36fbef8-3f03-40ce-b8c1-50d21e162c91/31ceb4ad-97ae-4994-9156-dc2819dfe7a6"
-					(reference "R9")
+					(reference "R22")
 					(unit 1)
 				)
@@
 		(dnp no)
 		(fields_autoplaced yes)
-		(property "Reference" "R7"
+		(property "Reference" "R21"
 			(at 114.935 83.1849 0)
 			(effects
@@
 			(project ""
 				(path "/e36fbef8-3f03-40ce-b8c1-50d21e162c91/31ceb4ad-97ae-4994-9156-dc2819dfe7a6"
-					(reference "R7")
+					(reference "R21")
 					(unit 1)
 				)
