File: design/RocketClock.kicad_pcb (KiCad board)
At the start: 2 copper layers, 100 x 100 mm, 124 parts, among them J1 PROG_CONN, J2 Right Output Conn, J3 Left Input Conn, P1 INPUT_PWR, Q1 SS8050, Q2 SS8050, Q3 MMBT3906, Q4 BC848W, Q5 BC848W, Q6 BC848W, Q7 BC848W, SW1 SW_Push, U1 TLV75533PDBV, U2 MAX7219, U3 TMP112xxDRL, U4 CH340G, U5 ATtiny84A-M, U6 ESP-12F, Y1 12MHz

Commit message: Update design and manufacturing files for v1.0.0 release
🤖 Generated with [Claude Code](https://claude.com/claude-code)

Co-Authored-By: Claude Opus 4.5 <noreply@anthropic.com>
Parts:
- removed D1: D_Schottky, Diode_SMD:D_SOD-123
- BZ1: value CBT-09427-SMT-TR -> KELIKING KLJ-9032-3627
- D66: value D_Schottky -> MBR0540T1G
- Y1: value 12MHz -> 12 MHz
- moved C9 1.90 mm to (123.8, 53.1), turned to 90 degrees
- turned Y1 to -90 degrees
Connections:
- P1 pad A4: /VUSB -> +5V
- P1 pad A9: /VUSB -> +5V
- P1 pad B4: /VUSB -> +5V
- P1 pad B9: /VUSB -> +5V
- Y1 pad 1: Net-(U4-XO) -> Net-(U4-XI)
- Y1 pad 2: Net-(U4-XI) -> GND
- Y1 pad 3: (no net) -> Net-(U4-XO)
- Y1 pad 4: (no net) -> GND
Routing:
- net /VUSB: track 18.2 -> 0.00 mm, vias 2 -> 0
- net +5V: track 117.1 -> 129.7 mm, vias 16 -> 18
- net Net-(U4-XI): track 7.30 -> 12.2 mm
- net GND: track 73.4 -> 74.9 mm
- net Net-(U4-XO): track 5.82 -> 5.24 mm
