File: design/usb_2_uart.kicad_sch (KiCad schematic)
At the start: 12 parts, among them Q1 SS8050, Q2 SS8050, U4 CH340G, Y1 12MHz

Commit message: Update design and manufacturing files for v1.0.0 release
🤖 Generated with [Claude Code](https://claude.com/claude-code)

Co-Authored-By: Claude Opus 4.5 <noreply@anthropic.com>
Parts:
- removed Y1: 12MHz, Crystal:Crystal_SMD_3225-4Pin_3.2x2.5mm_HandSoldering, symbol Device:Crystal
- added Y1: 12 MHz, Crystal:Crystal_SMD_3225-4Pin_3.2x2.5mm_HandSoldering, symbol Device:Crystal_GND24
Connections:
- net GND: now also Y1.2, Y1.4
- net at C9.1, U4.7 (XI): now also Y1.1
- net at C10.1, U4.8 (XO): now also Y1.3
Other:
- moved on the sheet: C10, C9
